Commit message: feat: update leg.urdf - add collision ball frame

File: config/leg.urdf (robot description, URDF)
Before this commit: robot el_mini, 5 links, 4 joints
Links:
- added link RF_HFE_CollBall, mass 0.0001; visual sphere radius=0.12
- added link RF_KFE_CollBall, mass 0.0001; visual sphere radius=0.12
Joints:
- added joint RF_HFE_Coll: type fixed, parent RF_HIP, child RF_HFE_CollBall, origin xyz=-0.02 -0.14999 -0.045056 rpy=3.1416 -1.5708 0, axis 0 0 1, limit lower=-0.5233 upper=3.14 effort=33.5 velocity=21
- added joint RF_KFE_Coll: type fixed, parent RF_THIGH, child RF_KFE_CollBall, origin xyz=0.13 0 -0.02 rpy=3.1416 0 1.5708, axis 0 0 1, limit lower=-0.6978 upper=3.925 effort=33.5 velocity=21
